File: 10knobs_mono_24bits/hardware/10knobs.kicad_pcb (KiCad board)
At the start: 2 copper layers, 44 parts, among them J1 3.3 GND, U1 MCP4822, U2 BluePill_STM32F103C, U3 6N138, U4 LM358

Commit message: Corrected schematic and PCB
Parts:
- J1: value 3.3 GND -> Conn_01x06_Female
Connections:
- C3 pad 1: Net-(C3-Pad1) -> +3V3
- R4 pad 1: Net-(C3-Pad1) -> +3V3
- U2 pad 18: Net-(C3-Pad1) -> +3V3
- U3 pad 8: Net-(C3-Pad1) -> +3V3
Routing:
- net +3V3: track 238.9 -> 292.4 mm, vias 0 -> 2
- net Net-(C3-Pad1): track 34.5 -> 0.00 mm

Commit message: Version 2.1, with correct MIDI and more stab cap
Parts:
- removed C3: 100n_tant, Capacitor_THT:CP_Radial_D5.0mm_P2.50mm
- removed TP6: IN2, TestPoint:TestPoint_THTPad_2.5x2.5mm_Drill1.2mm
- added C6: 100m chem, Capacitor_THT:CP_Radial_D5.0mm_P2.50mm, F.Cu at (74.5, 63.5)
- added C7: 0.1m ceram, Capacitor_THT:C_Disc_D3.0mm_W2.0mm_P2.50mm, F.Cu at (74.5, 69.5)
- C1: value 10m_chem -> 100m_chem
- C2: value 0.1micro_tantale -> 0.1m ceram; footprint Capacitor_THT:CP_Radial_D5.0mm_P2.50mm -> Capacitor_THT:C_Disc_D3.0mm_W2.0mm_P2.50mm
- moved R2 7.63 mm to (124.0, 63.5), turned to 180 degrees
- moved TP11 7.00 mm to (129.0, 62.5)
- moved TP4 4.98 mm to (56.0, 71.0)
Connections:
- J1 pad 2: (no net) -> Net-(J1-Pad2)
- J1 pad 6: (no net) -> Net-(J1-Pad6)
- U2 pad 1: (no net) -> Net-(U2-Pad1)
- U2 pad 15: (no net) -> Net-(U2-Pad15)
- U2 pad 17: (no net) -> Net-(U2-Pad17)
- U2 pad 2: (no net) -> Net-(U2-Pad2)
- U2 pad 23: (no net) -> Net-(U2-Pad23)
- U2 pad 28: (no net) -> Net-(U2-Pad28)
- U2 pad 29: (no net) -> Net-(U2-Pad29)
- U2 pad 3: (no net) -> Net-(U2-Pad3)
- U2 pad 30: (no net) -> Net-(U2-Pad30)
- U2 pad 31: (no net) -> Net-(U2-Pad31)
- U2 pad 32: (no net) -> Net-(U2-Pad32)
- U2 pad 33: (no net) -> Net-(U2-Pad33)
- U2 pad 34: (no net) -> Net-(U2-Pad34)
- U2 pad 35: (no net) -> Net-(U2-Pad35)
- U2 pad 36: (no net) -> Net-(U2-Pad36)
- U2 pad 37: (no net) -> Net-(U2-Pad37)
- U2 pad 4: (no net) -> Net-(U2-Pad4)
- U2 pad 41: (no net) -> Net-(U2-Pad41)
- U2 pad 42: (no net) -> Net-(U2-Pad42)
- U3 pad 1: (no net) -> Net-(U3-Pad1)
- U3 pad 4: (no net) -> Net-(U3-Pad4)
- U3 pad 7: (no net) -> Net-(U3-Pad7)
Routing:
- net GND: track 440.3 -> 493.2 mm, vias 0 -> 2
- net Net-(U1-Pad2): track 30.0 -> 76.1 mm
- net Net-(C1-Pad1): track 141.4 -> 105.6 mm
- net Net-(D1-Pad2): track 74.6 -> 45.4 mm
- net +3V3: track 292.4 -> 319.4 mm, vias 2 -> 0
- net Net-(R1-Pad2): track 61.3 -> 87.3 mm
- net Net-(R10-Pad2): track 11.8 -> 37.4 mm
- net Net-(RV2-Pad2): track 50.7 -> 44.4 mm
- net Net-(R8-Pad1): track 29.0 -> 34.9 mm
- net Net-(R2-Pad2): track 29.1 -> 34.8 mm
- net Net-(R2-Pad1): track 89.1 -> 84.3 mm
- net Net-(RV6-Pad2): track 34.1 -> 30.8 mm
- net Net-(J1-Pad1): track 23.8 -> 20.9 mm
- net Net-(RV11-Pad2): track 64.0 -> 61.5 mm
- net Net-(J1-Pad3): track 31.9 -> 29.8 mm
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