File: 10knobs_mono_24bits_MCP4822/hardware/10knobs.kicad_pcb (KiCad board)
At the start: 2 copper layers, 44 parts, among them J1 Conn_01x06_Female, U1 MCP4822, U2 BluePill_STM32F103C, U3 6N138, U4 LM358

Commit message: Changed name
Parts:
- moved TP7 2.50 mm to (138.5, 63.0)
Routing:
- net GND: track 0.00 -> 506.9 mm, vias 0 -> 2
- net +3V3: track 0.00 -> 336.2 mm
- net Net-(C1-Pad1): track 0.00 -> 108.9 mm
- net Net-(R1-Pad2): track 0.00 -> 88.5 mm
- net Net-(R2-Pad1): track 0.00 -> 88.0 mm
- net Net-(U1-Pad2): track 0.00 -> 78.9 mm
- net Net-(RV11-Pad2): track 0.00 -> 63.1 mm
- net Net-(RV8-Pad2): track 0.00 -> 59.3 mm
- net Net-(RV2-Pad2): track 0.00 -> 45.5 mm
- net Net-(D1-Pad2): track 0.00 -> 45.4 mm
- net Net-(RV5-Pad2): track 0.00 -> 42.8 mm
- net Net-(RV3-Pad2): track 0.00 -> 39.3 mm
- net Net-(RV10-Pad2): track 0.00 -> 38.3 mm
- net Net-(R10-Pad2): track 0.00 -> 37.4 mm
- net Net-(R2-Pad2): track 0.00 -> 35.6 mm
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- added copper zone on F.Cu, net GND
