File: 10knobs_mono_16bits_PT8211/hardware/10knobs_PT8211_complete1.kicad_pcb (KiCad board)
At the start: 2 copper layers, 47 parts, among them J1 GND, U1 PT8211, U2 BluePill_STM32F103C, U3 6N138, U4 LM358

Commit message: Completed mono PT8211 PCB
Routing:
- net GND: track 590.1 -> 587.6 mm
- net Net-(D1-Pad2): track 54.6 -> 55.4 mm
- net Net-(U1-Pad2): track 11.9 -> 12.6 mm
- net Net-(C9-Pad2): track 21.6 -> 20.9 mm
