File: 10knobs_mono_16bits_PT8211/hardware/10knobs_PT8211.sch (KiCad schematic (older format))
At the start: 48 parts, among them J1 Conn_01x06_Female, U1 PT8211, U2 BluePill_STM32F103C, U3 6N138, U4 LM358

Commit message: Removed auto saves
Parts:
- removed C3: 47u, Capacitor_THT:CP_Radial_D5.0mm_P2.50mm, symbol Device:CP
- U1: footprint Housings_SOIC:SOIC-8_3.9x4.9mm_Pitch1.27mm -> Package_SO:SOIC-8_3.9x4.9mm_P1.27mm
Connections:
- net GND: now also J1.1 (Pin_1), U2.39 (GND)
- net batt+: now also C1.1, C2.1
- net at U2.21 (PB12): no longer U1.2 (WS)
- net at U2.36 (PB8): now also U1.2 (WS)
Changed lines of the file:
@@
 EESchema Schematic File Version 4
+LIBS:10knobs_PT8211-cache
 EELAYER 26 0
 EELAYER END
@@
 Text GLabel 10400 5650 2    50   Input ~ 0
 DAC_out
-NoConn ~ 8350 4900
 Connection ~ 8500 2550
 Connection ~ 8750 2000
@@
 $EndComp
 Wire Wire Line
-	8650 5000 7850 5000
+	8650 5000 8400 5000
 Wire Wire Line
 	7850 5000 7850 5250
@@
 	0    -1   -1   0
 $EndComp
-Connection ~ 1550 4500
-Wire Wire Line
-	1550 4500 1550 4550
 Wire Wire Line
 	5200 2800 5700 2800
@@
 F 0 "U1" H 4600 7417 50  0000 C CNN
 F 1 "PT8211" H 4600 7326 50  0000 C CNN
-F 2 "Housings_SOIC:SOIC-8_3.9x4.9mm_Pitch1.27mm" H 4600 6900 50  0001 C CIN
+F 2 "Package_SO:SOIC-8_3.9x4.9mm_P1.27mm" H 4600 6900 50  0001 C CIN
 F 3 "" H 4600 6900 50  0001 C CNN
 	1    4600 6900
@@
 	4150 7150 4150 7200
 Wire Wire Line
-	6850 4900 6850 5550
-Wire Wire Line
 	3950 5550 3950 6800
 Wire Wire Line
 	3950 6800 4150 6800
-Wire Wire Line
-	3950 5550 6850 5550
 Wire Wire Line
 	6950 4900 6950 5450
@@
 	3800 7000 4150 7000
 NoConn ~ 5050 6800
-Wire Wire Line
-	5050 7150 5050 7350
 Wire Wire Line
 	5050 7550 4850 7550
@@
 $EndComp
 $Comp
-L Device:CP C3
-U 1 1 5FEF2E77
-P 5200 7350
-F 0 "C3" V 5455 7350 50  0000 C CNN
-F 1 "47u" V 5364 7350 50  0000 C CNN
-F 2 "Capacitor_THT:CP_Radial_D5.0mm_P2.50mm" H 5238 7200 50  0001 C CNN
-F 3 "~" H 5200 7350 50  0001 C CNN
-	1    5200 7350
-	0    -1   -1   0
-$EndComp
-Connection ~ 5050 7350
-Wire Wire Line
-	5050 7350 5050 7550
-$Comp
 L Device:C C8
 U 1 1 5FEF3075
@@
 $EndComp
 Connection ~ 5050 7550
-Wire Wire Line
-	5350 7350 5350 7450
 $Comp
 L power:GND #PWR0112
@@
 	0    -1   -1   0
 $EndComp
-Connection ~ 5350 7450
 Wire Wire Line
 	5350 7450 5350 7550
@@
 	5800 6350 6150 6350
 Connection ~ 6150 6350
+Connection ~ 1550 4500
+Wire Wire Line
+	1550 4500 1550 4550
+Text GLabel 1500 4550 0    50   Input ~ 0
+batt+
+Wire Wire Line
+	1550 4550 1500 4550
+$Comp
+L power:GND #PWR0114
+U 1 1 5FEB223F
+P 8400 5000
+F 0 "#PWR0114" H 8400 4750 50  0001 C CNN
+F 1 "GND" H 8405 4827 50  0000 C CNN
+F 2 "" H 8400 5000 50  0001 C CNN
+F 3 "" H 8400 5000 50  0001 C CNN
+	1    8400 5000
+	1    0    0    -1
+$EndComp
+Connection ~ 8400 5000
+Wire Wire Line
+	8400 5000 7850 5000
+Wire Wire Line
+	5050 7150 5050 7550
+Wire Wire Line
+	8350 4900 8350 5550
+Wire Wire Line
+	3950 5550 8350 5550
+NoConn ~ 6850 4900
 $EndSCHEMATC

Commit message: Adjusted lpf
Parts:
- C10: value 470p -> 680p
- R12, R6: value 7.5k -> 10k
Changed lines of the file:
@@
 P 5450 6650
 F 0 "R6" V 5243 6650 50  0000 C CNN
-F 1 "7.5k" V 5334 6650 50  0000 C CNN
+F 1 "10k" V 5334 6650 50  0000 C CNN
 F 2 "Resistor_THT:R_Axial_DIN0207_L6.3mm_D2.5mm_P7.62mm_Horizontal" V 5380 6650 50  0001 C CNN
 F 3 "~" H 5450 6650 50  0001 C CNN
@@
 P 5800 6650
 F 0 "R12" V 5593 6650 50  0000 C CNN
-F 1 "7.5k" V 5684 6650 50  0000 C CNN
+F 1 "10k" V 5684 6650 50  0000 C CNN
 F 2 "Resistor_THT:R_Axial_DIN0207_L6.3mm_D2.5mm_P7.62mm_Horizontal" V 5730 6650 50  0001 C CNN
 F 3 "~" H 5800 6650 50  0001 C CNN
@@
 P 5950 6800
 F 0 "C10" H 6065 6846 50  0000 L CNN
-F 1 "470p" H 6065 6755 50  0000 L CNN
+F 1 "680p" H 6065 6755 50  0000 L CNN
 F 2 "Capacitor_THT:C_Disc_D3.0mm_W2.0mm_P2.50mm" H 5988 6650 50  0001 C CNN
 F 3 "~" H 5950 6800 50  0001 C CNN

Commit message: Added a stab capacitor on the DAC
Parts:
- added C3: 1000uF, Capacitor_THT:CP_Radial_D7.5mm_P2.50mm, symbol Device:CP
Connections:
- net GND: now also C3.2
- net at C8.2, R2.1, U1.5 (VDD): now also C3.1
Changed lines of the file:
@@
 	8400 5000 7850 5000
 Wire Wire Line
-	5050 7150 5050 7550
+	5050 7150 5050 7250
 Wire Wire Line
 	8350 4900 8350 5550
@@
 	3950 5550 8350 5550
 NoConn ~ 6850 4900
+$Comp
+L Device:CP C3
+U 1 1 60AC718B
+P 5200 7250
+F 0 "C3" V 5455 7250 50  0000 C CNN
+F 1 "1000uF" V 5364 7250 50  0000 C CNN
+F 2 "Capacitor_THT:CP_Radial_D7.5mm_P2.50mm" H 5238 7100 50  0001 C CNN
+F 3 "~" H 5200 7250 50  0001 C CNN
+	1    5200 7250
+	0    -1   -1   0
+$EndComp
+Connection ~ 5050 7250
+Wire Wire Line
+	5050 7250 5050 7550
+Wire Wire Line
+	5350 7250 5350 7450
+Connection ~ 5350 7450
 $EndSCHEMATC
