File: 10knobs_mono_16bits_TDA1387/hardware/10knobs_TDA1387.sch (KiCad schematic (older format))
At the start: 52 parts, among them J1 Conn_01x06_Female, U2 BluePill_STM32F103C, U3 6N138, U4 LM358

Commit message: Finished routing
Parts:
- removed C2: 0.1u ceram, Capacitor_THT:C_Disc_D3.0mm_W2.0mm_P2.50mm, symbol Device:C
- removed C?: 1u, symbol Device:C
- removed C?: 10u, symbol Device:C
- removed C?: 1.5nF, symbol Device:C
- removed R?: R, symbol Device:R
- removed RV?: 1k - gain, symbol Device:R_POT
- removed U2: BluePill_STM32F103C, BluePill_breakouts:BluePill_STM32F103C, symbol bluepill_breakouts:BluePill_STM32F103C
- removed U4: LM358, Package_DIP:DIP-8_W7.62mm, symbol Amplifier_Operational:LM358
- removed U?: 2.7k, symbol Amplifier_Operational:TL072
- added C10: 1000p, Capacitor_THT:C_Disc_D5.0mm_W2.5mm_P2.50mm, symbol Device:C
- added C12: 680p, Capacitor_THT:C_Disc_D5.0mm_W2.5mm_P2.50mm, symbol Device:C
- added C13, C14: 100n, Capacitor_THT:C_Disc_D5.0mm_W2.5mm_P2.50mm, symbol Device:C
- added C9: 1u, Capacitor_THT:CP_Radial_D5.0mm_P2.50mm, symbol Device:CP
- added H1, H2, H3, H4: MountingHole, MountingHole:MountingHole_3.2mm_M3_ISO7380_Pad, symbol Mechanical:MountingHole
- added R12: 2.2k, Resistor_THT:R_Axial_DIN0207_L6.3mm_D2.5mm_P7.62mm_Horizontal, symbol Device:R
- added R6, R9: 10k, Resistor_THT:R_Axial_DIN0207_L6.3mm_D2.5mm_P7.62mm_Horizontal, symbol Device:R
- added SW1: SW_SPDT, Connector_PinSocket_2.54mm:PinSocket_1x03_P2.54mm_Vertical, symbol Switch:SW_SPDT
- added TP6: outRing, TestPoint:TestPoint_THTPad_2.5x2.5mm_Drill1.2mm, symbol Connector:TestPoint
- added U2: BluePill_STM32F103C_breadboard_friendly, BluePill:BluePill_STM32F103C_breadboard_friendly, symbol bluepill_breakouts:BluePill_STM32F103C_breadboard_friendly
- added unit 3 of U4
- added unit 2 of U4
- added U5: TL072, Package_DIP:DIP-8_W7.62mm_Socket_LongPads, symbol Amplifier_Operational:TL072
- C1: value 100u_chem -> 100u
- C11: renamed from C?; footprint (none) -> Capacitor_THT:CP_Radial_D5.0mm_P2.50mm
- RV9: renamed from RV?; value 10k - bias -> 1k - bias; footprint (none) -> Potentiometer_THT:Potentiometer_Bourns_3296W_Vertical
- TP7: value out1 -> outTip
- U1: renamed from U?; footprint Housings_SOIC:SOIC-8_3.9x4.9mm_Pitch1.27mm -> Package_SO:SO-8_3.9x4.9mm_P1.27mm
- U4: renamed from U?; footprint (none) -> Package_DIP:DIP-8_W7.62mm_Socket_LongPads
Connections:
- net +3V3: now also U2.18 (VCC3V3); no longer RV9.1
- net DAC_out: now also R12.1, U4.5 (+); no longer RV7.1
- net GND: now also C12.1, C13.2, C14.2, C9.2, U2.19 (GND), U2.20 (GND), U2.39 (GND), U4.4 (V-), U5.4 (V-)
- net batt+: now also RV9.1, C13.1, C14.1, U2.38 (5V_USB), U4.8 (V+), U5.8 (V+)
- net at RV3.2: now also U2.10 (PA5_SCK1)
- net at RV2.2: now also U2.11 (PA6_MISO1)
- net at RV1.2: now also U2.12 (PA7_MOSI1)
- net at RV11.2: now also U2.13 (PB0)
- net at RV10.2: now also U2.14 (PB1)
- net at R1.2, R4.2, U3.6 (VO2): now also U2.16 (PB11_SDA2)
- net at U1.1 (BCK): now also U2.22 (PB13_SCK2)
- net at U1.3 (DATA): now also U2.24 (PB15_MOSI2)
- net at D2.2 (A): now also U2.25 (PA8)
- net at J1.5 (Pin_5): now also U2.26 (PA9_TX1)
- net at J1.4 (Pin_4): now also U2.27 (PA10_RX1)
- net at U1.2 (WS): now also U2.36 (PB8)
- net at J1.3 (Pin_3): now also U2.40 (VCC3V3)
- net at R10.2, R11.2: now also U2.5 (PA0)
- net at RV8.2: now also U2.6 (PA1)
- net at RV6.2: now also U2.7 (PA2_TX2)
- net at RV5.2: now also U2.8 (PA3_RX2)
- net at RV4.2: now also U2.9 (PA4)
- net at R8.1, RV7.2: now also U5.5 (+)
- net at C5.1, TP7.1: now also SW1.3 (C)
- net at C4.1: now also U5.6 (-), U5.7
- net at U1.7 (REF): now also C9.1
- net at U1.8 (RCH): now also U4.2 (-), R12.2
- new net: R9.2, U4.6 (-), U4.7
- new net: C12.2, R6.2, U5.3 (+)
- new net: SW1.2 (B), TP6.1
- new net: C10.1, R6.1, R9.1
- new net filter_out: C10.2, RV7.1, U5.1, U5.2 (-)
- no-connect marks 23 -> 22
