File: 10knobs_mono_16bits_TDA1387/hardware/10knobs_TDA1387.kicad_pcb (KiCad board)
At the start: 2 copper layers, 48 parts, among them J1 Conn_01x06_Female, U1 PT8211, U2 BluePill_STM32F103C, U3 6N138, U4 LM358

Commit message: Finished routing
Parts:
- removed C2: 0.1u ceram, Capacitor_THT:C_Disc_D3.0mm_W2.0mm_P2.50mm
- added C11: 10u, Capacitor_THT:CP_Radial_D5.0mm_P2.50mm, F.Cu at (121.9, 96.6)
- added C12: 680p, Capacitor_THT:C_Disc_D5.0mm_W2.5mm_P2.50mm, F.Cu at (123.4, 77.3)
- added C13: 100n, Capacitor_THT:C_Disc_D5.0mm_W2.5mm_P2.50mm, F.Cu at (105.9, 82.4)
- added C14: 100n, Capacitor_THT:C_Disc_D5.0mm_W2.5mm_P2.50mm, F.Cu at (139.4, 87.2)
- added H1: MountingHole, MountingHole:MountingHole_3.2mm_M3_ISO7380_Pad, F.Cu at (48.6, 22.4)
- added H2: MountingHole, MountingHole:MountingHole_3.2mm_M3_ISO7380_Pad, F.Cu at (48.6, 95.6)
- added H3: MountingHole, MountingHole:MountingHole_3.2mm_M3_ISO7380_Pad, F.Cu at (137.7, 22.2)
- added H4: MountingHole, MountingHole:MountingHole_3.2mm_M3_ISO7380_Pad, F.Cu at (137.5, 95.6)
- added RV9: 1k - bias, Potentiometer_THT:Potentiometer_Bourns_3296W_Vertical, F.Cu at (111.5, 95.5)
- added SW1: SW_SPDT, Connector_PinSocket_2.54mm:PinSocket_1x03_P2.54mm_Vertical, F.Cu at (129.5, 64.9)
- added TP6: outRing, TestPoint:TestPoint_THTPad_2.5x2.5mm_Drill1.2mm, F.Cu at (129.7, 60.3)
- added U5: TL072, Package_DIP:DIP-8_W7.62mm_Socket_LongPads, F.Cu at (134.5, 81.8)
- C1: value 100u_chem -> 100u
- C10: value 680p -> 1000p; footprint Capacitor_THT:C_Disc_D3.0mm_W2.0mm_P2.50mm -> Capacitor_THT:C_Disc_D5.0mm_W2.5mm_P2.50mm
- C9: value 1000p -> 1u; footprint Capacitor_THT:C_Disc_D3.0mm_W2.0mm_P2.50mm -> Capacitor_THT:CP_Radial_D5.0mm_P2.50mm
- J1: value Conn_01x06_Female -> Prog - GND
- R12: value 10k -> 2.2k
- R9: value 100R -> 10k
- TP7: value out1 -> outTip
- U1: value PT8211 -> TDA1387; footprint Package_SO:SOIC-8_3.9x4.9mm_P1.27mm -> Package_SO:SO-8_3.9x4.9mm_P1.27mm
- U2: value BluePill_STM32F103C -> BluePill_STM32F103C_breadboard_friendly; footprint BluePill_breakouts:BluePill_STM32F103C -> BluePill:BluePill_STM32F103C_breadboard_friendly
- U4: value LM358 -> TL072; footprint Package_DIP:DIP-8_W7.62mm -> Package_DIP:DIP-8_W7.62mm_Socket_LongPads
- moved C1 31.3 mm to (90.9, 65.0), turned to 0 degrees
- moved C9 29.3 mm to (100.6, 78.7), turned to 0 degrees
- moved U3 26.5 mm to (60.6, 73.9), turned to 270 degrees
- moved D1 25.4 mm to (64.4, 65.7), turned to 180 degrees
- moved U4 23.6 mm to (109.2, 85.0), turned to 90 degrees
- moved R2 19.7 mm to (89.7, 77.2), turned to 0 degrees
- moved U1 19.2 mm to (84.2, 80.8)
- moved R1 19.0 mm to (53.1, 63.1), turned to 270 degrees
- moved R8 18.7 mm to (123.4, 89.5), turned to 90 degrees
- moved C8 18.2 mm to (80.0, 81.9)
- moved R11 13.3 mm to (101.8, 64.6), turned to 0 degrees
- moved C4 12.9 mm to (138.4, 77.1)
- moved C5 12.8 mm to (138.2, 68.7)
- moved R10 12.8 mm to (101.7, 67.8), turned to 0 degrees
- moved C10 12.1 mm to (130.6, 68.7), turned to 0 degrees
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Connections:
- C10 pad 2: GND -> /filter_out
- C9 pad 1: DAC_out -> Net-(C9-Pad1)
- C9 pad 2: Net-(C9-Pad2) -> GND
- J1 pad 2: (no net) -> Net-(J1-Pad2)
- J1 pad 6: (no net) -> Net-(J1-Pad6)
- R12 pad 1: Net-(C10-Pad1) -> DAC_out
- R12 pad 2: Net-(C9-Pad2) -> Net-(R12-Pad2)
- R6 pad 1: Net-(C9-Pad2) -> Net-(C10-Pad1)
- R6 pad 2: Net-(R6-Pad2) -> Net-(C12-Pad2)
- R9 pad 1: Net-(C5-Pad1) -> Net-(C10-Pad1)
- RV7 pad 1: DAC_out -> /filter_out
- TP7 pad 1: Net-(R9-Pad2) -> Net-(C5-Pad1)
- U1 pad 6: (no net) -> Net-(U1-Pad6)
- U1 pad 7: (no net) -> Net-(C9-Pad1)
- U1 pad 8: Net-(R6-Pad2) -> Net-(R12-Pad2)
- U2 pad 1: (no net) -> Net-(U2-Pad1)
- U2 pad 15: (no net) -> Net-(U2-Pad15)
- U2 pad 17: (no net) -> Net-(U2-Pad17)
- U2 pad 2: (no net) -> Net-(U2-Pad2)
- U2 pad 21: (no net) -> Net-(U2-Pad21)
- U2 pad 23: (no net) -> Net-(U2-Pad23)
- U2 pad 28: (no net) -> Net-(U2-Pad28)
- U2 pad 29: (no net) -> Net-(U2-Pad29)
- U2 pad 3: (no net) -> Net-(U2-Pad3)
- U2 pad 30: (no net) -> Net-(U2-Pad30)
- U2 pad 31: (no net) -> Net-(U2-Pad31)
- U2 pad 32: (no net) -> Net-(U2-Pad32)
- U2 pad 33: (no net) -> Net-(U2-Pad33)
- U2 pad 34: (no net) -> Net-(U2-Pad34)
- U2 pad 35: (no net) -> Net-(U2-Pad35)
- U2 pad 37: (no net) -> Net-(U2-Pad37)
- U2 pad 4: (no net) -> Net-(U2-Pad4)
- U3 pad 1: (no net) -> Net-(U3-Pad1)
- U3 pad 4: (no net) -> Net-(U3-Pad4)
- U3 pad 7: (no net) -> Net-(U3-Pad7)
- U4 pad 2: DAC_out -> Net-(R12-Pad2)
- U4 pad 3: Net-(C10-Pad1) -> Net-(C11-Pad2)
- U4 pad 5: Net-(R8-Pad1) -> DAC_out
- U4 pad 6: Net-(C4-Pad1) -> Net-(R9-Pad2)
- U4 pad 7: Net-(C4-Pad1) -> Net-(R9-Pad2)
Routing:
- net GND: track 594.4 -> 671.6 mm, vias 0 -> 4
- net batt+: track 154.3 -> 216.0 mm
- net Net-(R12-Pad2): track 0.00 -> 48.1 mm, vias 0 -> 2
- net Net-(D1-Pad2): track 54.6 -> 15.6 mm
- net Net-(C12-Pad2): track 0.00 -> 36.1 mm
- net /filter_out: track 0.00 -> 31.5 mm
- net Net-(D1-Pad1): track 16.1 -> 45.7 mm
- net Net-(C11-Pad2): track 0.00 -> 26.1 mm
- net DAC_out: track 42.5 -> 16.6 mm
- net Net-(R8-Pad1): track 31.0 -> 56.4 mm
- net Net-(C10-Pad1): track 14.7 -> 38.6 mm
- net Net-(U1-Pad1): track 39.5 -> 17.3 mm
- net Net-(C9-Pad2): track 21.6 -> 0.00 mm
- net Net-(RV5-Pad2): track 38.0 -> 58.9 mm
- net Net-(U1-Pad3): track 27.4 -> 7.54 mm
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Other:
- net class Default: clearance 0.25 -> 0.23; via_dia 2.3 -> 2; via_drill 1.2 -> 1
- rule trace_clearance: 0.25 -> 0.23
- board text added: "TDA1387"
- board text added: "TES - 10k synth - TDA1387 - 5 patch diam 1mm"

Commit message: Updated PCB
Routing:
- net batt+: track 216.0 -> 217.5 mm
- net Net-(RV6-Pad2): track 21.9 -> 21.2 mm
- net Net-(C3-Pad1): track 22.3 -> 22.9 mm
