File: 10knobs_mono_16bits_TDA1387/hardware/10knobs_TDA1387.kicad_pcb (KiCad board)
At the start: 2 copper layers, 59 parts, among them J1 Prog - GND, SW1 SW_SPDT, U1 TDA1387, U2 BluePill_STM32F103C_breadboar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, U3 6N138, U4 TL072, U5 TL072

Commit message: Moved to seperate folders
Other:
- net class Default removed
- net class easy removed
